File: pcb_esp.sch (KiCad schematic (older format))
At the start: 32 parts, among them J1 CONN_01X07, J2 CONN_01X03, J3 CONN_01X17, Q1 S8050, Q2 S8050, U1 LP38691, U2 ESP-12E, U3 ET024002DMU

Commit message: smd transistors + minor changes
transistors changed to smd
programming header changed to angled
minor routing and 3d model alignment changes
Parts:
- J1: footprint Pin_Headers:Pin_Header_Straight_1x07_Pitch2.54mm -> Pin_Headers:Pin_Header_Angled_1x07_Pitch2.54mm
- Q1, Q2: footprint TO_SOT_Packages_THT:TO-92_Molded_Narrow -> TO_SOT_Packages_SMD:SOT-23_Handsoldering; symbol S8050 -> BC817
Changed lines of the file:
@@
 Connection ~ 5500 1550
 Wire Wire Line
-	7150 2250 5500 2250
+	5500 2250 7150 2250
 Wire Wire Line
 	6800 2250 6800 2000
@@
 F 0 "J1" H 9981 5742 50  0000 L CNN
 F 1 "CONN_01X07" H 9981 5649 50  0000 L CNN
-F 2 "Pin_Headers:Pin_Header_Straight_1x07_Pitch2.54mm" H 9900 5700 50  0001 C CNN
+F 2 "Pin_Headers:Pin_Header_Angled_1x07_Pitch2.54mm" H 9900 5700 50  0001 C CNN
 F 3 "" H 9900 5700 50  0001 C CNN
 	1    9900 5700
-	1    0    0    -1
+	1    0    0    1
 $EndComp
 Wire Wire Line
@@
 	7150 1550 7150 1700
 Wire Wire Line
-	7150 2000 7150 2250
+	7150 2250 7150 2000
 Connection ~ 6800 2250
 Wire Wire Line
@@
 Buttons
 $Comp
-L S8050 Q1
+L BC817 Q1
 U 1 1 596EFC1D
 P 1950 4000
 F 0 "Q1" H 2141 4047 50  0000 L CNN
 F 1 "S8050" H 2141 3954 50  0000 L CNN
-F 2 "TO_SOT_Packages_THT:TO-92_Molded_Narrow" H 2150 3925 50  0001 L CIN
+F 2 "TO_SOT_Packages_SMD:SOT-23_Handsoldering" H 2150 3925 50  0001 L CIN
 F 3 "" H 1950 4000 50  0001 L CNN
 	1    1950 4000
@@
 $EndComp
 $Comp
-L S8050 Q2
+L BC817 Q2
 U 1 1 596EFD25
 P 1950 4700
 F 0 "Q2" H 2141 4653 50  0000 L CNN
 F 1 "S8050" H 2141 4746 50  0000 L CNN
-F 2 "TO_SOT_Packages_THT:TO-92_Molded_Narrow" H 2150 4625 50  0001 L CIN
+F 2 "TO_SOT_Packages_SMD:SOT-23_Handsoldering" H 2150 4625 50  0001 L CIN
 F 3 "" H 1950 4700 50  0001 L CNN
 	1    1950 4700
